File: Hardware/KiCad Project/TempMonitor.sch (KiCad schematic (older format))
At the start: 38 parts, among them M1 SMD-RES-10K-1%-1_8W_0805_, M2 SMD-RES-10K-1%-1_8W_0805_, M3 SMD-RES-10K-1%-1_8W_0805_, M4 SMD-RES-10K-1%-1_8W_0805_, M5 SMD-RES-10K-1%-1_8W_0805_, M6 SMD-RES-10K-1%-1_8W_0805_, M7 SMD-RES-10K-1%-1_8W_0805_, M8 SMD-RES-10K-1%-1_8W_0805_, M9 SMD-RES-10K-1%-1_8W_0805_, P1 Pad, P10 Pad, P11 Pad, P2 ProgrammingPad, P3 Pad, P4 Pad, P5 Pad, P6 Pad, P7 Pad, P8 Pad, P9 Pad, U1 DRIVER-TM1637_SOP20_, U2 LED-4-BETY-7-SEG_2X7P-30X14MM_, U3 LED-4-BETY-7-SEG_2X7P-30X14MM_, U4 LED-4-BETY-7-SEG_2X7P-30X14MM_, U5 LED-4-BETY-7-SEG_2X7P-30X14MM_, U6 DRIVER-TM1637_SOP20_, U7 DRIVER-TM1637_SOP20_, U8 DRIVER-TM1637_SOP20_, U9 ATMEGA16U2-MU, Y1 SMD-CRYSTAL-16MHZ-8PF-20PPM-4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

Commit message: Update
Gerber files added, BOM added, PCB redone, separate clock traces for
led-drivers made.
Parts:
- renumbered C4 to C2, C2 to C3, C3 to C4, P11 to P10, P2 to P11, P3 to P2, P5 to P3, P6 to P5, P7 to P6, P8 to P7, P9 to P8, P10 to P9, M2 to R1, M1 to R10, R1 to R11, M3 to R2, M4 to R3, M5 to R4, M6 to R5, M7 to R6, M8 to R7, M9 to R8, R2 to R9, U2 to U1, U1 to U2, U6 to U4, U9 to U5, U4 to U6, U5 to U8, U8 to U9
Connections:
- net CLK1: now also U2.18 (CLK)
- net CLK2: now also U4.18 (CLK)
- net CLK3: now also U7.18 (CLK)
- net CLK4: now also U9.18 (CLK)
- removed net CLK: U2.18 (CLK), U4.18 (CLK), U7.18 (CLK), U9.18 (CLK)
Other:
- moved on the sheet: R7, R8
