File: Hardware/Version 2/tempmonitor.sch (EAGLE design)
At the start: 41 parts, among them IC1 74LS595D, IC2 74LS595D, IC3 74LS595D, IC4 74LS595D, IC5 74LS595D, J2 TP_8, J3 USB-MICROB, T1 NPN, T2 NPN, T3 NPN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

Commit message: Version 1.0
Parts:
- D1, D2: value 3.6V -> 16V; device SparkFun-DiscreteSemi:DIODE-ZENER3.3V -> SparkFun-DiscreteSemi:DIODE-ZENER16V
- RN1, RN2, RN3, RN4, RN5, RN6, RN7, RN8: device resistor-dil:4R-NEXBS8V -> resistor-dil:4R-NEXBV8V
Changed lines of the file:
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@@
 <grid distance="0.1" unitdist="inch" unit="inch" style="lines" multiple="1" display="no" altdistance="0.01" altunitdist="inch" altunit="inch"/>
 <layers>
-<layer number="1" name="Top" color="4" fill="1" visible="no" active="no"/>
-<layer number="16" name="Bottom" color="1" fill="1" visible="no" active="no"/>
-<layer number="17" name="Pads" color="2" fill="1" visible="no" active="no"/>
-<layer number="18" name="Vias" color="2" fill="1" visible="no" active="no"/>
-<layer number="19" name="Unrouted" color="6" fill="1" visible="no" active="no"/>
-<layer number="20" name="Dimension" color="15" fill="1" visible="no" active="no"/>
-<layer number="21" name="tPlace" color="7" fill="1" visible="no" active="no"/>
-<layer number="22" name="bPlace" color="7" fill="1" visible="no" active="no"/>
-<layer number="23" name="tOrigins" color="15" fill="1" visible="no" active="no"/>
-<layer number="24" name="bOrigins" color="15" fill="1" visible="no" active="no"/>
-<layer number="25" name="tNames" color="7" fill="1" visible="no" active="no"/>
-<layer number="26" name="bNames" color="7" fill="1" visible="no" active="no"/>
-<layer number="27" name="tValues" color="7" fill="1" visible="no" active="no"/>
-<layer number="28" name="bValues" color="7" fill="1" visible="no" active="no"/>
+<layer number="1" name="Top" color="4" fill="1" visible="yes" active="no"/>
+<layer number="16" name="Bottom" color="1" fill="1" visible="yes" active="no"/>
+<layer number="17" name="Pads" color="2" fill="1" visible="yes" active="no"/>
+<layer number="18" name="Vias" color="2" fill="1" visible="yes" active="no"/>
+<layer number="19" name="Unrouted" color="6" fill="1" visible="yes" active="no"/>
+<layer number="20" name="Dimension" color="15" fill="1" visible="yes" active="no"/>
+<layer number="21" name="tPlace" color="7" fill="1" visible="yes" active="no"/>
+<layer number="22" name="bPlace" color="7" fill="1" visible="yes" active="no"/>
+<layer number="23" name="tOrigins" color="15" fill="1" visible="yes" active="no"/>
+<layer number="24" name="bOrigins" color="15" fill="1" visible="yes" active="no"/>
+<layer number="25" name="tNames" color="7" fill="1" visible="yes" active="no"/>
+<layer number="26" name="bNames" color="7" fill="1" visible="yes" active="no"/>
+<layer number="27" name="tValues" color="7" fill="1" visible="yes" active="no"/>
+<layer number="28" name="bValues" color="7" fill="1" visible="yes" active="no"/>
 <layer number="29" name="tStop" color="7" fill="3" visible="no" active="no"/>
 <layer number="30" name="bStop" color="7" fill="6" visible="no" active="no"/>
@@
 <layer number="35" name="tGlue" color="7" fill="4" visible="no" active="no"/>
 <layer number="36" name="bGlue" color="7" fill="5" visible="no" active="no"/>
-<layer number="37" name="tTest" color="7" fill="1" visible="no" active="no"/>
-<layer number="38" name="bTest" color="7" fill="1" visible="no" active="no"/>
+<layer number="37" name="tTest" color="7" fill="1" visible="yes" active="no"/>
+<layer number="38" name="bTest" color="7" fill="1" visible="yes" active="no"/>
 <layer number="39" name="tKeepout" color="4" fill="11" visible="no" active="no"/>
 <layer number="40" name="bKeepout" color="1" fill="11" visible="no" active="no"/>
@@
 <layer number="44" name="Drills" color="7" fill="1" visible="no" active="no"/>
 <layer number="45" name="Holes" color="7" fill="1" visible="no" active="no"/>
-<layer number="46" name="Milling" color="3" fill="1" visible="no" active="no"/>
-<layer number="47" name="Measures" color="7" fill="1" visible="no" active="no"/>
-<layer number="48" name="Document" color="7" fill="1" visible="no" active="no"/>
-<layer number="49" name="Reference" color="7" fill="1" visible="no" active="no"/>
-<layer number="50" name="dxf" color="7" fill="1" visible="no" active="no"/>
-<layer number="51" name="tDocu" color="7" fill="1" visible="no" active="no"/>
-<layer number="52" name="bDocu" color="7" fill="1" visible="no" active="no"/>
-<layer number="53" name="tGND_GNDA" color="7" fill="9" visible="no" active="no"/>
-<layer number="54" name="bGND_GNDA" color="1" fill="9" visible="no" active="no"/>
-<layer number="56" name="wert" color="7" fill="1" visible="no" active="no"/>
-<layer number="57" name="tCAD" color="7" fill="1" visible="no" active="no"/>
-<layer number="59" name="tCarbon" color="7" fill="1" visible="no" active="no"/>
-<layer number="60" name="bCarbon" color="7" fill="1" visible="no" active="no"/>
+<layer number="46" name="Milling" color="3" fill="1" visible="yes" active="no"/>
+<layer number="47" name="Measures" color="7" fill="1" visible="yes" active="no"/>
+<layer number="48" name="Document" color="7" fill="1" visible="yes" active="no"/>
+<layer number="49" name="Reference" color="7" fill="1" visible="yes" active="no"/>
+<layer number="50" name="dxf" color="7" fill="1" visible="yes" active="no"/>
+<layer number="51" name="tDocu" color="7" fill="1" visible="yes" active="no"/>
+<layer number="52" name="bDocu" color="7" fill="1" visible="yes" active="no"/>
+<layer number="53" name="tGND_GNDA" color="7" fill="9" visible="yes" active="no"/>
+<layer number="54" name="bGND_GNDA" color="1" fill="9" visible="yes" active="no"/>
+<layer number="56" name="wert" color="7" fill="1" visible="yes" active="no"/>
+<layer number="57" name="tCAD" color="7" fill="1" visible="yes" active="no"/>
+<layer number="59" name="tCarbon" color="7" fill="1" visible="yes" active="no"/>
+<layer number="60" name="bCarbon" color="7" fill="1" visible="yes" active="no"/>
 <layer number="90" name="Modules" color="5" fill="1" visible="yes" active="yes"/>
 <layer number="91" name="Nets" color="2" fill="1" visible="yes" active="yes"/>
@@
 <part name="R1" library="resistor" deviceset="R-EU_" device="R0805W" value="68 ohm"/>
 <part name="R2" library="resistor" deviceset="R-EU_" device="R0805W" value="68 ohm"/>
-<part name="D1" library="SparkFun-DiscreteSemi" deviceset="DIODE-ZENER" device="3.3V" value="3.6V"/>
-<part name="D2" library="SparkFun-DiscreteSemi" deviceset="DIODE-ZENER" device="3.3V" value="3.6V"/>
+<part name="D1" library="SparkFun-DiscreteSemi" deviceset="DIODE-ZENER" device="16V" value="16V"/>
+<part name="D2" library="SparkFun-DiscreteSemi" deviceset="DIODE-ZENER" device="16V" value="16V"/>
 <part name="R3" library="resistor" deviceset="R-EU_" device="R0805W" value="2.2k ohm"/>
 <part name="GND5" library="supply1" deviceset="GND" device=""/>
 <part name="P+7" library="supply1" deviceset="+5V" device=""/>
 <part name="P+8" library="supply1" deviceset="+5V" device=""/>
-<part name="RN1" library="resistor-dil" deviceset="4R-N" device="EXBS8V" value="560 ohm"/>
+<part name="RN1" library="resistor-dil" deviceset="4R-N" device="EXBV8V" value="560 ohm"/>
 <part name="GND6" library="supply1" deviceset="GND" device=""/>
 <part name="P+9" library="supply1" deviceset="+5V" device=""/>
@@
 <part name="GND7" library="supply1" deviceset="GND" device=""/>
 <part name="IC2" library="SparkFun-DigitalIC" deviceset="74*595" device="D" technology="LS"/>
-<part name="RN2" library="resistor-dil" deviceset="4R-N" device="EXBS8V" value="560 ohm"/>
+<part name="RN2" library="resistor-dil" deviceset="4R-N" device="EXBV8V" value="560 ohm"/>
 <part name="GND3" library="supply1" deviceset="GND" device=""/>
 <part name="P+3" library="supply1" deviceset="+5V" device=""/>
 <part name="P+4" library="supply1" deviceset="+5V" device=""/>
-<part name="RN3" library="resistor-dil" deviceset="4R-N" device="EXBS8V" value="560 ohm"/>
+<part name="RN3" library="resistor-dil" deviceset="4R-N" device="EXBV8V" value="560 ohm"/>
 <part name="LED2" library="display-kingbright" deviceset="B?56-12*WA" device="C" technology="Y"/>
 <part name="IC1" library="SparkFun-DigitalIC" deviceset="74*595" device="D" technology="LS"/>
-<part name="RN4" library="resistor-dil" deviceset="4R-N" device="EXBS8V" value="560 ohm"/>
+<part name="RN4" library="resistor-dil" deviceset="4R-N" device="EXBV8V" value="560 ohm"/>
 <part name="GND4" library="supply1" deviceset="GND" device=""/>
 <part name="P+5" library="supply1" deviceset="+5V" device=""/>
 <part name="P+6" library="supply1" deviceset="+5V" device=""/>
-<part name="RN5" library="resistor-dil" deviceset="4R-N" device="EXBS8V" value="560 ohm"/>
+<part name="RN5" library="resistor-dil" deviceset="4R-N" device="EXBV8V" value="560 ohm"/>
 <part name="LED3" library="display-kingbright" deviceset="B?56-12*WA" device="C" technology="Y"/>
 <part name="IC3" library="SparkFun-DigitalIC" deviceset="74*595" device="D" technology="LS"/>
-<part name="RN6" library="resistor-dil" deviceset="4R-N" device="EXBS8V" value="560 ohm"/>
+<part name="RN6" library="resistor-dil" deviceset="4R-N" device="EXBV8V" value="560 ohm"/>
 <part name="C1" library="SparkFun-Capacitors" deviceset="CAP_POL" device="F80" value="10uF"/>
 <part name="J2" library="TempMonitor" deviceset="TP_8" device=""/>
@@
 <part name="P+11" library="supply1" deviceset="+5V" device=""/>
 <part name="P+12" library="supply1" deviceset="+5V" device=""/>
-<part name="RN7" library="resistor-dil" deviceset="4R-N" device="EXBS8V" value="560 ohm"/>
+<part name="RN7" library="resistor-dil" deviceset="4R-N" device="EXBV8V" value="560 ohm"/>
 <part name="LED4" library="display-kingbright" deviceset="B?56-12*WA" device="C" technology="Y"/>
 <part name="IC5" library="SparkFun-DigitalIC" deviceset="74*595" device="D" technology="LS"/>
-<part name="RN8" library="resistor-dil" deviceset="4R-N" device="EXBS8V" value="560 ohm"/>
+<part name="RN8" library="resistor-dil" deviceset="4R-N" device="EXBV8V" value="560 ohm"/>
 <part name="R7" library="resistor" deviceset="R-EU_" device="R0805W" value="10k"/>
 <part name="P+13" library="supply1" deviceset="+5V" device=""/>
