File: Hardware/Version 2/Temp monitor.brd (EAGLE design)
At the start: 99 x 49 mm, 41 parts, among them IC1 74LS595D, IC2 74LS595D, IC3 74LS595D, IC4 74LS595D, IC5 74LS595D, J2 TP_8, J3 USB-MICROB, T1 NPN, T2 NPN, T3 NPN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

Commit message: Added schematic in PDF
Parts:
- D1, D2: value 16V -> 3.6V
Connections:
- net N$6 renamed DISPLAY_DATA
Changed lines of the file:
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@@
 <?xml version="1.0" encoding="utf-8"?>
 <!DOCTYPE eagle SYSTEM "eagle.dtd">
-<eagle version="7.6.0">
+<eagle version="7.7.0">
 <drawing>
 <settings>
@@
 </autorouter>
 <elements>
-<element name="D1" library="SparkFun-DiscreteSemi" package="SOD-123" value="16V" x="18.5276" y="8.3914" smashed="yes" rot="MR90">
+<element name="D1" library="SparkFun-DiscreteSemi" package="SOD-123" value="3.6V" x="18.5276" y="8.3914" smashed="yes" rot="MR90">
 <attribute name="PROD_ID" value="DIO-12440" x="18.5276" y="8.3914" size="1.778" layer="28" rot="MR90" display="off"/>
 <attribute name="NAME" x="18.1212" y="10.779" size="1.016" layer="26" rot="MR90"/>
 </element>
-<element name="D2" library="SparkFun-DiscreteSemi" package="SOD-123" value="16V" x="12.2722" y="8.52" smashed="yes" rot="MR90">
+<element name="D2" library="SparkFun-DiscreteSemi" package="SOD-123" value="3.6V" x="12.2722" y="8.52" smashed="yes" rot="MR90">
 <attribute name="PROD_ID" value="DIO-12440" x="12.2722" y="8.52" size="1.778" layer="28" rot="MR90" display="off"/>
 <attribute name="NAME" x="11.9928" y="10.806" size="1.016" layer="26" rot="MR90"/>
@@
 <wire x1="15.7244" y1="33.5677" x2="15.9678" y2="33.3243" width="0.4064" layer="16"/>
 </signal>
-<signal name="N$6">
-<contactref element="IC4" pad="9"/>
+<signal name="DISPLAY_DATA">
 <contactref element="IC2" pad="14"/>
-<wire x1="11.9144" y1="42.1084" x2="11.9144" y2="45.162" width="0.4064" layer="16"/>
 <wire x1="11.9144" y1="45.162" x2="11.931" y2="45.162" width="0.4064" layer="16"/>
 <via x="11.931" y="45.162" extent="1-16" drill="0.6"/>
@@
 <wire x1="33.14" y1="45.162" x2="33.14" y2="42.2644" width="0.4064" layer="16"/>
 <wire x1="33.14" y1="42.2644" x2="33.1744" y2="42.2644" width="0.4064" layer="16"/>
+<contactref element="IC4" pad="9"/>
+<wire x1="11.9144" y1="45.162" x2="11.9144" y2="42.1084" width="0.4064" layer="16"/>
 </signal>
 <signal name="N$34">
