File: Hardware/Version 2/Temp monitor.sch (EAGLE design)
At the start: 41 parts, among them IC1 74LS595D, IC2 74LS595D, IC3 74LS595D, IC4 74LS595D, IC5 74LS595D, J2 TP_8, J3 USB-MICROB, T1 NPN, T2 NPN, T3 NPN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

Commit message: Added schematic in PDF
Parts:
- D1, D2: value 16V -> 3.6V
Connections:
- net N$6 renamed DISPLAY_DATA
Other:
- note added: "CONTROL CIRCUIT"
- note added: "DISPLAY ANODE DRIVERS"
- note added: "DISPLAY CATHODE DRIVER"
- note added: "Temp monitor UF"
- moved on the sheet: C1, C2, C3, C4, C5, C6, D1, D2, IC1, IC2, IC3, IC4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
